Commit message: imu added

File: robot_urdf_description/inertia.xacro (robot description, xacro)
@@ -30,3 +30,12 @@
     </inertial>
 </xacro:macro>
+<xacro:macro name="imu_inertia" params="mass x y z *origin">
+    <inertial>
+        <xacro:insert_block name="origin"/>
+        <mass value="${mass}"/>
+        <inertia ixx="${(1.0/12.0) * mass * (y * y + z * z)}" ixy="0.0" ixz="0.0"
+                 iyy="${(1.0/12.0) * mass * (x * x + z * z)}" iyz="0.0"
+                 izz="${(1.0/12.0) * mass * (x * x + y * y)}"/>
+    </inertial>
+</xacro:macro>
 </robot>

File: robot_urdf_description/robot_main_urdf.xacro (robot description, xacro)
@@ -6,4 +6,5 @@
     <xacro:include filename="lidar_sensor.xacro"/>
     <xacro:include filename="camera_sensor.xacro"/>
+    <xacro:include filename="imu.xacro"/>
     <!--<xacro:include filename="depth_camera_sensor.xacro"/>-->
 </robot>
